File: pcb-left/Alipt-Keyboard-Left.kicad_pcb (KiCad board)
At the start: 2 copper layers, 195 x 119.6 mm, 83 parts, among them J1 LED, J2 4PIN, J3 OLED, P1 i2c_pin, P2 i2c_pin, SW0 SW_PUSH, SW1 SW_PUSH, SW10 SW_PUSH, SW11 SW_PUSH, SW12 SW_PUSH, SW13 SW_PUSH, SW14 SW_PUSH, SW15 SW_PUSH, SW16 SW_PUSH, SW17 SW_PUSH, SW18 SW_PUSH, SW19 SW_PUSH, SW2 SW_PUSH, SW20 SW_PUSH, SW21 SW_PUSH, SW22 SW_PUSH, SW23 SW_PUSH, SW24 SW_PUSH, SW25 SW_PUSH, SW26 SW_PUSH, SW27 SW_PUSH, SW28 SW_PUSH, SW29 SW_PUSH, SW3 SW_PUSH, SW30 SW_PUSH, SW31 SW_PUSH, SW32 Rotary_Encoder_Switch, SW4 SW_PUSH, SW5 SW_PUSH, SW6 SW_PUSH, SW7 SW_PUSH, SW8 SW_PUSH, SW9 SW_PUSH, U1 ProMicro

Commit message: revision 1 complete pcbs
Parts:
- moved D22 16.5 mm to (95.9, 117.3), turned to 90 degrees
- moved D30 15.3 mm to (177.4, 149.2), turned to 78 degrees
- moved D28 14.8 mm to (59.6, 136.4), turned to 90 degrees
- moved D25 11.8 mm to (155.6, 124.8), turned to 78 degrees
- moved D29 9.89 mm to (134.0, 141.3), turned to 78 degrees
- moved D24 8.72 mm to (136.8, 120.8), turned to 78 degrees
- moved D8 8.45 mm to (88.0, 79.2), turned to 90 degrees
- moved D14 8.40 mm to (60.0, 77.0), turned to 90 degrees
- moved D4 8.19 mm to (162.8, 67.9), turned to 78 degrees
- moved D3 8.17 mm to (144.2, 63.8), turned to 78 degrees
- moved D23 8.13 mm to (117.5, 117.3), turned to 90 degrees
- moved D7 8.08 mm to (63.9, 58.0), turned to 90 degrees
- moved D27 8.05 mm to (192.9, 133.2), turned to 78 degrees
- moved D9 8.04 mm to (111.4, 79.2), turned to 90 degrees
- moved D12 7.96 mm to (168.1, 88.9), turned to 78 degrees
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Routing:
- net row4: track 71.4 -> 274.2 mm
- net row3: track 66.4 -> 245.7 mm
- net row2: track 68.4 -> 240.0 mm
- net row1: track 71.0 -> 213.2 mm
- net row0: track 73.0 -> 209.5 mm
- net col1: track 77.4 -> 203.5 mm
- net col4: track 147.2 -> 271.6 mm
- net col2: track 100.0 -> 208.7 mm
- net col3: track 121.8 -> 218.2 mm
- net col0: track 56.5 -> 141.1 mm
- net col5: track 171.8 -> 240.6 mm
- net SW32A: track 232.9 -> 298.4 mm
- net Net-(D30-Pad2): track 0.00 -> 25.1 mm
- net Net-(D22-Pad2): track 0.00 -> 22.7 mm
- net Net-(D29-Pad2): track 0.00 -> 16.3 mm
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Other:
- board size 195 x 119.6 mm -> 197.4 x 119.6 mm

Commit message: update
Parts:
- added SW302: SW_PUSH, cftkb:SW_Cherry_MX1A_2.00u_PCBNOSCREEN, F.Cu at (160.3, 136.1)
- added SW312: SW_PUSH, cftkb:SW_Cherry_MX1A_1.25u_PCBNOSCREEN, F.Cu at (190.7, 142.6)
- W1: moved to B.Cu
- moved J2 61.7 mm to (202.1, 43.2), turned to 0 degrees
- moved W1 51.2 mm to (206.4, 44.1), turned to 180 degrees
- moved P2 44.7 mm to (199.6, 58.4), turned to 270 degrees
- moved P1 41.1 mm to (202.6, 58.4), turned to 270 degrees
- moved D32 37.5 mm to (204.4, 146.2)
- moved SW32 37.5 mm to (215.1, 150.1)
- moved RSW1 16.0 mm to (214.2, 83.4), turned to 0 degrees
- moved TH1 12.3 mm to (188.3, 50.9)
- moved R1 12.2 mm to (208.3, 84.8), turned to 90 degrees
- moved R2 10.4 mm to (210.8, 84.8), turned to 90 degrees
- moved J1 8.03 mm to (205.7, 81.9)
- moved U1 5.45 mm to (217.0, 61.7)
- moved J3 4.79 mm to (213.4, 80.1)
Routing:
- net row0: track 209.5 -> 153.0 mm, vias 0 -> 1
- net SW32A: track 298.4 -> 351.0 mm, vias 4 -> 2
- net DATA: track 73.9 -> 22.9 mm, vias 2 -> 1
- net row4: track 274.2 -> 245.6 mm, vias 0 -> 1
- net ENCA: track 85.1 -> 113.5 mm, vias 2 -> 0
- net ENCB: track 79.7 -> 105.9 mm, vias 2 -> 1
- net LED: track 79.7 -> 65.9 mm, vias 3 -> 1
- net row1: track 213.2 -> 199.6 mm, vias 0 -> 1
- net col0: track 141.1 -> 129.1 mm, vias 2 -> 0
- net col1: track 203.5 -> 215.1 mm, vias 2 -> 0
- net col5: track 240.6 -> 229.2 mm, vias 2 -> 0
- net row2: track 240.0 -> 251.2 mm, vias 0 -> 1
- net GND: track 44.4 -> 55.5 mm, vias 3 -> 9
- net col2: track 208.7 -> 215.7 mm, vias 2 -> 0
- net /i2c_d: track 27.6 -> 22.5 mm
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Other:
- board size 197.4 x 119.6 mm -> 192.3 x 119.6 mm
