File: pcb-left/Alipt-Keyboard-Left.sch (KiCad schematic (older format))
At the start: 83 parts, among them J1 LED, J2 4PIN, J3 OLED, P1 i2c_pin, P2 i2c_pin, SW0 SW_PUSH, SW1 SW_PUSH, SW10 SW_PUSH, SW11 SW_PUSH, SW12 SW_PUSH, SW13 SW_PUSH, SW14 SW_PUSH, SW15 SW_PUSH, SW16 SW_PUSH, SW17 SW_PUSH, SW18 SW_PUSH, SW19 SW_PUSH, SW2 SW_PUSH, SW20 SW_PUSH, SW21 SW_PUSH, SW22 SW_PUSH, SW23 SW_PUSH, SW24 SW_PUSH, SW25 SW_PUSH, SW26 SW_PUSH, SW27 SW_PUSH, SW28 SW_PUSH, SW29 SW_PUSH, SW3 SW_PUSH, SW30 SW_PUSH, SW31 SW_PUSH, SW32 Rotary_Encoder_Switch, SW4 SW_PUSH, SW5 SW_PUSH, SW6 SW_PUSH, SW7 SW_PUSH, SW8 SW_PUSH, SW9 SW_PUSH, U1 ProMicro

Commit message: update
Parts:
- added SW302: SW_PUSH, cftkb:SW_Cherry_MX1A_2.00u_PCBNOSCREEN, symbol SofleKeyboard-rescue:SW_PUSH-Lily58-cache-Lily58_Pro-rescue
- added SW312: SW_PUSH, cftkb:SW_Cherry_MX1A_1.25u_PCBNOSCREEN, symbol SofleKeyboard-rescue:SW_PUSH-Lily58-cache-Lily58_Pro-rescue
Connections:
- net col1: now also SW312.1
- net col2: now also SW302.1
- net at D30.2 (A), SW30.2: now also SW302.2
- net at D31.2 (A), SW31.2: now also SW312.2
Changed lines of the file:
@@
 Wire Wire Line
 	10150 3950 10950 3950
-Wire Wire Line
-	9550 3650 9550 4300
 Connection ~ 9350 4600
 Wire Wire Line
@@
 Wire Wire Line
 	2550 4950 2750 4950
+$Comp
+L SofleKeyboard-rescue:SW_PUSH-Lily58-cache-Lily58_Pro-rescue SW302
+U 1 1 5F796447
+P 9050 4800
+F 0 "SW302" H 9050 4950 50  0000 C CNN
+F 1 "SW_PUSH" H 9050 4700 50  0000 C CNN
+F 2 "cftkb:SW_Cherry_MX1A_2.00u_PCBNOSCREEN" H 9050 4800 50  0001 C CNN
+F 3 "" H 9050 4800 50  0000 C CNN
+	1    9050 4800
+	1    0    0    -1
+$EndComp
+Wire Wire Line
+	9350 4800 9500 4800
+Wire Wire Line
+	9500 4800 9500 4300
+Wire Wire Line
+	9500 4300 9350 4300
+Connection ~ 9350 4300
+Wire Wire Line
+	8750 4300 8750 4800
+Connection ~ 8750 4300
+$Comp
+L SofleKeyboard-rescue:SW_PUSH-Lily58-cache-Lily58_Pro-rescue SW312
+U 1 1 5F7A102F
+P 9850 4750
+F 0 "SW312" H 9850 4900 50  0000 C CNN
+F 1 "SW_PUSH" H 9850 4650 50  0000 C CNN
+F 2 "cftkb:SW_Cherry_MX1A_1.25u_PCBNOSCREEN" H 9850 4750 50  0001 C CNN
+F 3 "" H 9850 4750 50  0000 C CNN
+	1    9850 4750
+	1    0    0    -1
+$EndComp
+Wire Wire Line
+	9550 3650 9550 4300
+Connection ~ 9550 4300
+Wire Wire Line
+	9550 4300 9550 4750
+Wire Wire Line
+	10150 4750 10350 4750
+Wire Wire Line
+	10350 4750 10350 4300
+Wire Wire Line
+	10350 4300 10150 4300
+Connection ~ 10150 4300
 $EndSCHEMATC
